File: poi_PCB/_autosave-poi_PCB.sch (KiCad schematic (older format))
At the start: 41 parts, among them J4 USB_C_Receptacle_USB2.0, Q3 Q_NMOS_DGS, SW1 SW_Push, U1 ESP32-WROOM-32D, U2 CH340C, U3 AMS1117-3.3, U6 MH-CD42

Commit message: Verified reset circuit
Breadboarded and edited reset circuit.
-USBC port moved closer to center
-transistors replaced because of issues with transistor quality
Parts:
- R2: LCSC (none) -> C25091
Changed lines of the file:
@@
 F 2 "Resistor_SMD:R_0402_1005Metric" H 4650 5000 50  0001 C CNN
 F 3 "~" H 4650 5000 50  0001 C CNN
+F 4 "C25091" H 4650 5000 50  0001 C CNN "LCSC"
 	1    4650 5000
 	0    1    1    0
