File: poi_PCB/_autosave-poi_PCB.sch (KiCad schematic (older format))
At the start: 69 parts, among them J4 USB_C_Receptacle_USB2.0, Q1 AO4407C, Q2 AO3400A, Q3 AO3400A, Q4 AO3400A, Q5 AO4407C, SW3 TL2233OA, U1 ESP32-WROOM-32D, U2 CH340C, U3 AMS1117-3.3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

Commit message: updated sourcing info
Parts:
- D2, D3, D4, D5, D6, D7, D8, D9: LCSC C139127 -> (none); MANUFACTURER (none) -> Aliexpress
- H1, H2, H3, TP1, TP2: MANUFACTURER (none) -> NA
- J4, SW3: MANUFACTURER (none) -> Digikey
- MK1: MANUFACTURER CUI Devices -> Local
- U1, U6: MANUFACTURER (none) -> Local
- U2: MANUFACTURER (none) -> Aliexpress
- U3: LCSC C6186 -> (none); MANUFACTURER (none) -> Local
- U4: MANUFACTURER STMicroelectronics -> LCSC
Changed lines of the file:
@@
 F 2 "LED_SMD:LED_WS2812B_PLCC4_5.0x5.0mm_P3.2mm" H 7650 850 50  0001 L TNN
 F 3 "https://cdn-shop.adafruit.com/datasheets/WS2812B.pdf" H 7700 775 50  0001 L TNN
-F 4 "C139127" H 7600 1150 50  0001 C CNN "LCSC"
+F 4 "" H 7600 1150 50  0001 C CNN "LCSC"
+F 5 "Aliexpress" H 7600 1150 50  0001 C CNN "MANUFACTURER"
 	1    7600 1150
 	1    0    0    -1
@@
 F 2 "LED_SMD:LED_WS2812B_PLCC4_5.0x5.0mm_P3.2mm" H 8550 850 50  0001 L TNN
 F 3 "https://cdn-shop.adafruit.com/datasheets/WS2812B.pdf" H 8600 775 50  0001 L TNN
-F 4 "C139127" H 8500 1150 50  0001 C CNN "LCSC"
+F 4 "" H 8500 1150 50  0001 C CNN "LCSC"
+F 5 "Aliexpress" H 8500 1150 50  0001 C CNN "MANUFACTURER"
 	1    8500 1150
 	1    0    0    -1
@@
 F 2 "LED_SMD:LED_WS2812B_PLCC4_5.0x5.0mm_P3.2mm" H 9500 850 50  0001 L TNN
 F 3 "https://cdn-shop.adafruit.com/datasheets/WS2812B.pdf" H 9550 775 50  0001 L TNN
-F 4 "C139127" H 9450 1150 50  0001 C CNN "LCSC"
+F 4 "" H 9450 1150 50  0001 C CNN "LCSC"
+F 5 "Aliexpress" H 9450 1150 50  0001 C CNN "MANUFACTURER"
 	1    9450 1150
 	1    0    0    -1
@@
 F 2 "LED_SMD:LED_WS2812B_PLCC4_5.0x5.0mm_P3.2mm" H 10400 850 50  0001 L TNN
 F 3 "https://cdn-shop.adafruit.com/datasheets/WS2812B.pdf" H 10450 775 50  0001 L TNN
-F 4 "C139127" H 10350 1150 50  0001 C CNN "LCSC"
+F 4 "" H 10350 1150 50  0001 C CNN "LCSC"
+F 5 "Aliexpress" H 10350 1150 50  0001 C CNN "MANUFACTURER"
 	1    10350 1150
 	1    0    0    -1
@@
 F 2 "LED_SMD:LED_WS2812B_PLCC4_5.0x5.0mm_P3.2mm" H 7650 2250 50  0001 L TNN
 F 3 "https://cdn-shop.adafruit.com/datasheets/WS2812B.pdf" H 7700 2175 50  0001 L TNN
-F 4 "C139127" H 7600 2550 50  0001 C CNN "LCSC"
+F 4 "" H 7600 2550 50  0001 C CNN "LCSC"
+F 5 "Aliexpress" H 7600 2550 50  0001 C CNN "MANUFACTURER"
 	1    7600 2550
 	1    0    0    -1
@@
 F 2 "LED_SMD:LED_WS2812B_PLCC4_5.0x5.0mm_P3.2mm" H 8550 2250 50  0001 L TNN
 F 3 "https://cdn-shop.adafruit.com/datasheets/WS2812B.pdf" H 8600 2175 50  0001 L TNN
-F 4 "C139127" H 8500 2550 50  0001 C CNN "LCSC"
+F 4 "" H 8500 2550 50  0001 C CNN "LCSC"
+F 5 "Aliexpress" H 8500 2550 50  0001 C CNN "MANUFACTURER"
 	1    8500 2550
 	1    0    0    -1
@@
 F 2 "LED_SMD:LED_WS2812B_PLCC4_5.0x5.0mm_P3.2mm" H 9500 2250 50  0001 L TNN
 F 3 "https://cdn-shop.adafruit.com/datasheets/WS2812B.pdf" H 9550 2175 50  0001 L TNN
-F 4 "C139127" H 9450 2550 50  0001 C CNN "LCSC"
+F 4 "" H 9450 2550 50  0001 C CNN "LCSC"
+F 5 "Aliexpress" H 9450 2550 50  0001 C CNN "MANUFACTURER"
 	1    9450 2550
 	1    0    0    -1
@@
 F 2 "LED_SMD:LED_WS2812B_PLCC4_5.0x5.0mm_P3.2mm" H 10400 2250 50  0001 L TNN
 F 3 "https://cdn-shop.adafruit.com/datasheets/WS2812B.pdf" H 10450 2175 50  0001 L TNN
-F 4 "C139127" H 10350 2550 50  0001 C CNN "LCSC"
+F 4 "" H 10350 2550 50  0001 C CNN "LCSC"
+F 5 "Aliexpress" H 10350 2550 50  0001 C CNN "MANUFACTURER"
 	1    10350 2550
 	1    0    0    -1
@@
 F 2 "Package_TO_SOT_SMD:SOT-223-3_TabPin2" H 3800 7250 50  0001 C CNN
 F 3 "http://www.advanced-monolithic.com/pdf/ds1117.pdf" H 3900 6800 50  0001 C CNN
-F 4 "C6186" H 3800 7050 50  0001 C CNN "LCSC"
+F 4 "" H 3800 7050 50  0001 C CNN "LCSC"
+F 5 "Local" H 3800 7050 50  0001 C CNN "MANUFACTURER"
 	1    3800 7050
 	1    0    0    -1
@@
 F 2 "TestPoint:TestPoint_THTPad_D3.0mm_Drill1.5mm" H 6650 6800 50  0001 C CNN
 F 3 "~" H 6650 6800 50  0001 C CNN
+F 4 "NA" H 6450 6800 50  0001 C CNN "MANUFACTURER"
 	1    6450 6800
 	-1   0    0    1
@@
 F 2 "Package_SO:SOIC-16_3.9x9.9mm_P1.27mm" H 5850 5400 50  0001 L CNN
 F 3 "https://datasheet.lcsc.com/szlcsc/Jiangsu-Qin-Heng-CH340C_C84681.pdf" H 5450 6750 50  0001 C CNN
+F 4 "Aliexpress" H 5800 5950 50  0001 C CNN "MANUFACTURER"
 	1    5800 5950
 	0    -1   -1   0
@@
 F 2 "MountingHole:MountingHole_3.2mm_M3" H 7200 3950 50  0001 C CNN
 F 3 "~" H 7200 3950 50  0001 C CNN
+F 4 "NA" H 7200 3950 50  0001 C CNN "MANUFACTURER"
 	1    7200 3950
 	1    0    0    -1
@@
 F 2 "MountingHole:MountingHole_3.2mm_M3" H 7200 4150 50  0001 C CNN
 F 3 "~" H 7200 4150 50  0001 C CNN
+F 4 "NA" H 7200 4150 50  0001 C CNN "MANUFACTURER"
 	1    7200 4150
 	1    0    0    -1
@@
 F 2 "MountingHole:MountingHole_3.2mm_M3" H 7200 4350 50  0001 C CNN
 F 3 "~" H 7200 4350 50  0001 C CNN
+F 4 "NA" H 7200 4350 50  0001 C CNN "MANUFACTURER"
 	1    7200 4350
 	1    0    0    -1
@@
 F 2 "RF_Module:ESP32-WROOM-32" H 2000 3850 50  0001 C CNN
 F 3 "https://www.espressif.com/sites/default/files/documentation/esp32-wroom-32d_esp32-wroom-32u_datasheet_en.pdf" H 1700 5400 50  0001 C CNN
+F 4 "Local" H 2000 5350 50  0001 C CNN "MANUFACTURER"
 	1    2000 5350
 	1    0    0    -1
@@
 F 2 "USB4120-03-C_REVA:GCT_USB4120-03-C_REVA" H 6150 3750 50  0001 C CNN
 F 3 "https://www.usb.org/sites/default/files/documents/usb_type-c.zip" H 6150 3750 50  0001 C CNN
+F 4 "Digikey" H 6000 3750 50  0001 C CNN "MANUFACTURER"
 	1    6000 3750
 	0    1    1    0
@@
 F 4 "6" H 10100 4250 50  0001 L BNN "PARTREV"
 F 5 "IPC-7351B" H 10100 4250 50  0001 L BNN "STANDARD"
-F 6 "STMicroelectronics" H 10100 4250 50  0001 L BNN "MANUFACTURER"
+F 6 "LCSC" H 10100 4250 50  0001 L BNN "MANUFACTURER"
 	1    10100 4250
 	1    0    0    -1
@@
 F 5 "1.0" H 9450 5900 50  0001 L BNN "PARTREV"
 F 6 "Manufacturer Recommendations" H 9450 5900 50  0001 L BNN "STANDARD"
-F 7 "CUI Devices" H 9450 5900 50  0001 L BNN "MANUFACTURER"
+F 7 "Local" H 9450 5900 50  0001 L BNN "MANUFACTURER"
 	1    9450 5900
 	1    0    0    -1
@@
 F 2 "Arduino:MH-CD42" H 5450 8000 50  0001 C CNN
 F 3 "" H 5450 8000 50  0001 C CNN
+F 4 "Local" H 5500 7250 50  0001 C CNN "MANUFACTURER"
 	1    5500 7250
 	1    0    0    -1
@@
 F 2 "TestPoint:TestPoint_Loop_D1.80mm_Drill1.0mm_Beaded" H 5300 7450 50  0001 C CNN
 F 3 "~" H 5300 7450 50  0001 C CNN
+F 4 "NA" H 5100 7450 50  0001 C CNN "MANUFACTURER"
 	1    5100 7450
 	1    0    0    -1
@@
 F 2 "TL2233OA:TL2233OA" H 3200 3000 50  0001 C CNN
 F 3 "~" H 3200 3000 50  0001 C CNN
+F 4 "Digikey" H 3200 2800 50  0001 C CNN "MANUFACTURER"
 	1    3200 2800
 	1    0    0    -1
