File: poi_PCB/poi_PCB.sch (KiCad schematic (older format))
At the start: 41 parts, among them J4 USB_C_Receptacle_USB2.0, Q3 Q_NMOS_DGS, SW1 SW_Push, U1 ESP32-WROOM-32D, U2 CH340C, U3 AMS1117-3.3, U6 MH-CD42

Commit message: redone traces, changed accelerometer, supercapacitor and mic
Parts:
- removed SW1: SW_Push, Button_Switch_SMD:SW_SPST_TL3342, symbol Switch:SW_Push
- added C13, C15, C2: .1uF, Capacitor_SMD:C_0402_1005Metric, symbol Device:C_Small
- added C3: 220pF, Capacitor_SMD:C_0402_1005Metric, symbol Device:C_Small
- added C4: CP1_Small, Capacitor_THT:CP_Radial_D13.0mm_P5.00mm, symbol Device:CP1_Small
- added D1: LED, LED_SMD:LED_0603_1608Metric, symbol Device:LED
- added MK1: CMM-4030D-261-I2S-TR, CMM-4030D-261-I2S-TR:MIC_CMM-4030D-261-I2S-TR, symbol CMM-4030D-261-I2S-TR:CMM-4030D-261-I2S-TR
- added Q1, Q5: AO4407C, Package_SO:SOIC-8_3.9x4.9mm_P1.27mm, symbol Transistor_FET:FDS9435A
- added Q2, Q4: AO3400A, Package_TO_SOT_SMD:SOT-23, symbol Device:Q_NMOS_DGS
- added R11, R13, R17, R18, R19, R20, R21: 10K, Resistor_SMD:R_0402_1005Metric, symbol Device:R_Small_US
- added R5: 220R, Resistor_SMD:R_0402_1005Metric, symbol Device:R_Small_US
- added R7, R8, R9: 51R, Resistor_SMD:R_0603_1608Metric, symbol Device:R_Small_US
- added SW3: TL2233OA, TL2233OA:TL2233OA, symbol TL2233OA:TL2233OA
- added TP1: 5V_EN_L, TestPoint:TestPoint_Loop_D1.80mm_Drill1.0mm_Beaded, symbol Connector:TestPoint_Small
- added U4: LSM6DS33TR, LSM6DS33TR:PQFN50P300X300X86-16N, symbol LSM6DS33TR:LSM6DS33TR
- D10: value D_Schottky_Small -> 1N5819WS; footprint Diode_SMD:D_SMA -> Diode_SMD:D_SOD-323; LCSC C22452 -> C191023
- Q3: value Q_NMOS_DGS -> AO3400A; LCSC C8545 -> C20917
- R2: LCSC (none) -> C25091
- TP2: renamed from +BATT1; value TestPoint -> +BAT
Connections:
- net labels added: 5V_EN_L, BCLK, CHARGE_CAP_EN, CS, D_OUT_I2S, FIRE, SCL, SDA, SHIELD, WS
- wire segments 120 -> 171
Other:
- note added: "Accelerometer\n"
- note added: "Capacitor charge\n"
- note added: "ESP32\n"
- note added: "Filtering capacitors for LED matrix"
- note added: "MEMS Microphone"
- note added: "Place accelerometer \nnear mounting hole"
- note added: "USB-C port"
- note added: "battery charge controller and 5V boost converter\n"
- note added: "capacitor discharge\n"
- moved on the sheet: C1, C10, C11, C12, C14, C16, C17, C18, C5, C6, C7, C8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

Commit message: Verified pinouts
-Pinouts all checked to be compatible with peripherals.
-FIRE is pulled up to +CAP, and drains within 20 minutes if the device is turned off
Parts:
- added R12: 10K, Resistor_SMD:R_0402_1005Metric, symbol Device:R_Small_US
- added R16, R22, R23: 100K, Resistor_SMD:R_0402_1005Metric, symbol Device:R_Small_US
- R1: value 10K -> 1K
- R21: value 10K -> 100K
Connections:
- net +3V3: now also U4.5 (CS), R12.1; no longer R21.1
- net +BATT: now also R16.1
- net BCLK: now also U1.11 (IO26); no longer U1.26 (IO4)
- net CHARGE_CAP_EN: now also U1.12 (IO27)
- net D_OUT_I2S: now also U1.9 (IO33); no longer U1.30 (IO18)
- net GND: now also R21.2, R23.2; no longer R17.1
- net SCL: now also U1.26 (IO4)
- net SDA: now also U1.27 (IO16)
- net WS: now also U1.10 (IO25); no longer U1.29 (IO5)
- net FIRE_L: now reaches U1.13 (IO14)
- net FIRE_L: now also Q4.2 (G), R17.1
- net CAP_VSENSE: now reaches U1.14 (IO12)
- net CAP_VSENSE: now also R22.2, R23.1
- net BAT_VSENSE: now reaches U1.6 (IO34)
- net BAT_VSENSE: now also R21.1, R16.2
- net at C4.1, Q1.5 (D), Q1.6 (D)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: now also R17.2, R22.1
- net SDO: now reaches U4.4 (SDO/SA0)
- net SDO: now also R12.2
- removed net CS: R21.2, U4.5 (CS)
- removed net FIRE: Q4.2 (G), R17.2
Other:
- moved on the sheet: D1, R17, R5, TP1, TP2
Changed lines of the file:
@@
 L power:+BATT #PWR0111
 U 1 1 6193F7FC
-P 6500 7250
-F 0 "#PWR0111" H 6500 7100 50  0001 C CNN
-F 1 "+BATT" H 6515 7423 50  0000 C CNN
-F 2 "" H 6500 7250 50  0001 C CNN
-F 3 "" H 6500 7250 50  0001 C CNN
-	1    6500 7250
+P 6450 6800
+F 0 "#PWR0111" H 6450 6650 50  0001 C CNN
+F 1 "+BATT" H 6465 6973 50  0000 C CNN
+F 2 "" H 6450 6800 50  0001 C CNN
+F 3 "" H 6450 6800 50  0001 C CNN
+	1    6450 6800
 	1    0    0    -1
 $EndComp
@@
 L Connector:TestPoint TP2
 U 1 1 61A595F3
-P 6500 7250
-F 0 "TP2" H 6558 7368 50  0000 L CNN
-F 1 "+BAT" H 6558 7277 50  0000 L CNN
-F 2 "TestPoint:TestPoint_THTPad_D3.0mm_Drill1.5mm" H 6700 7250 50  0001 C CNN
-F 3 "~" H 6700 7250 50  0001 C CNN
-	1    6500 7250
+P 6450 6800
+F 0 "TP2" H 6508 6918 50  0000 L CNN
+F 1 "+BAT" H 6508 6827 50  0000 L CNN
+F 2 "TestPoint:TestPoint_THTPad_D3.0mm_Drill1.5mm" H 6650 6800 50  0001 C CNN
+F 3 "~" H 6650 6800 50  0001 C CNN
+	1    6450 6800
 	-1   0    0    1
 $EndComp
@@
 Wire Wire Line
 	7850 6000 8000 6000
-Text Label 2600 4650 0    50   ~ 0
-WS
-Text Label 2600 4550 0    50   ~ 0
-BCLK
-Text Label 2600 5350 0    50   ~ 0
-D_OUT_I2S
 $Comp
 L Device:LED D1
 U 1 1 61AE6CB7
-P 3050 4850
-F 0 "D1" H 3043 4595 50  0000 C CNN
-F 1 "LED" H 3043 4686 50  0000 C CNN
-F 2 "LED_SMD:LED_0603_1608Metric" H 3050 4850 50  0001 C CNN
-F 3 "~" H 3050 4850 50  0001 C CNN
-	1    3050 4850
+P 3400 4850
+F 0 "D1" H 3393 4595 50  0000 C CNN
+F 1 "LED" H 3393 4686 50  0000 C CNN
+F 2 "LED_SMD:LED_0603_1608Metric" H 3400 4850 50  0001 C CNN
+F 3 "~" H 3400 4850 50  0001 C CNN
+	1    3400 4850
 	-1   0    0    1
 $EndComp
@@
 L Device:R_Small_US R5
 U 1 1 61AE7FCD
-P 2800 4850
-F 0 "R5" V 2595 4850 50  0000 C CNN
-F 1 "220R" V 2686 4850 50  0000 C CNN
-F 2 "Resistor_SMD:R_0402_1005Metric" H 2800 4850 50  0001 C CNN
-F 3 "~" H 2800 4850 50  0001 C CNN
-	1    2800 4850
+P 3150 4850
+F 0 "R5" V 2945 4850 50  0000 C CNN
+F 1 "220R" V 3036 4850 50  0000 C CNN
+F 2 "Resistor_SMD:R_0402_1005Metric" H 3150 4850 50  0001 C CNN
+F 3 "~" H 3150 4850 50  0001 C CNN
+	1    3150 4850
 	0    1    1    0
 $EndComp
@@
 L power:GND #PWR0130
 U 1 1 61AE94F1
-P 3200 4850
-F 0 "#PWR0130" H 3200 4600 50  0001 C CNN
-F 1 "GND" V 3205 4722 50  0000 R CNN
-F 2 "" H 3200 4850 50  0001 C CNN
-F 3 "" H 3200 4850 50  0001 C CNN
-	1    3200 4850
+P 3550 4850
+F 0 "#PWR0130" H 3550 4600 50  0001 C CNN
+F 1 "GND" V 3555 4722 50  0000 R CNN
+F 2 "" H 3550 4850 50  0001 C CNN
+F 3 "" H 3550 4850 50  0001 C CNN
+	1    3550 4850
 	0    -1   -1   0
 $EndComp
@@
 P 5050 3600
 F 0 "R1" H 5118 3646 50  0000 L CNN
-F 1 "10K" H 5118 3555 50  0000 L CNN
+F 1 "1K" H 5118 3555 50  0000 L CNN
 F 2 "Resistor_SMD:R_0402_1005Metric" V 5090 3590 50  0001 C CNN
 F 3 "~" H 5050 3600 50  0001 C CNN
@@
 	10450 5800 10400 5800
 Wire Wire Line
-	2700 4850 2600 4850
-Wire Wire Line
 	2000 3950 2000 3700
 Wire Notes Line
@@
 SHIELD
 Text Label 3150 1300 2    50   ~ 0
-FIRE
-Wire Wire Line
-	3150 1500 3150 1300
+FIRE_L
 Wire Wire Line
 	3450 1550 3450 1500
-Wire Wire Line
-	3350 1500 3450 1500
-$Comp
-L Device:R_Small_US R17
-U 1 1 61B52924
-P 3250 1500
-F 0 "R17" V 3045 1500 50  0000 C CNN
-F 1 "10K" V 3136 1500 50  0000 C CNN
-F 2 "Resistor_SMD:R_0402_1005Metric" H 3250 1500 50  0001 C CNN
-F 3 "~" H 3250 1500 50  0001 C CNN
-	1    3250 1500
-	0    1    -1   0
-$EndComp
 $Comp
 L power:GND #PWR0145
@@
 capacitor discharge\n
 Wire Wire Line
-	2150 1300 2750 1300
+	2150 1300 2550 1300
 Wire Wire Line
 	2750 1300 2750 700
 Wire Wire Line
-	2750 700  4050 700
+	2750 700  3150 700
 Wire Wire Line
 	4050 700  4050 850
@@
 	1    0    0    -1
 $EndComp
-$Comp
-L Device:R_Small_US R21
-U 1 1 61AC45F4
-P 9150 3900
-F 0 "R21" H 9218 3946 50  0000 L CNN
-F 1 "10K" H 9218 3855 50  0000 L CNN
-F 2 "Resistor_SMD:R_0402_1005Metric" H 9150 3900 50  0001 C CNN
-F 3 "~" H 9150 3900 50  0001 C CNN
-	1    9150 3900
-	1    0    0    -1
-$EndComp
 Wire Wire Line
 	8550 3800 8850 3800
@@
 Wire Wire Line
 	8850 3800 8850 3750
-Wire Wire Line
-	8850 3800 9150 3800
 Text Label 9500 4450 2    50   ~ 0
 CS
@@
 Text Label 8850 4100 0    50   ~ 0
 SCL
-Text Label 9150 4100 0    50   ~ 0
+Text Label 9150 3800 0    50   ~ 0
 CS
-Wire Wire Line
-	9150 4100 9150 4000
 Wire Wire Line
 	8850 4100 8850 4000
@@
 	1    0    0    -1
 $EndComp
-Connection ~ 3450 1500
 Connection ~ 2150 1300
 Connection ~ 1850 1100
@@
 L Connector:TestPoint_Small TP1
 U 1 1 61AFE2F0
-P 6350 6800
-F 0 "TP1" H 6398 6846 50  0000 L CNN
-F 1 "5V_EN_L" H 6398 6755 50  0000 L CNN
-F 2 "TestPoint:TestPoint_Loop_D1.80mm_Drill1.0mm_Beaded" H 6550 6800 50  0001 C CNN
-F 3 "~" H 6550 6800 50  0001 C CNN
-	1    6350 6800
+P 5100 7450
+F 0 "TP1" H 5148 7496 50  0000 L CNN
+F 1 "5V_EN_L" H 5148 7405 50  0000 L CNN
+F 2 "TestPoint:TestPoint_Loop_D1.80mm_Drill1.0mm_Beaded" H 5300 7450 50  0001 C CNN
+F 3 "~" H 5300 7450 50  0001 C CNN
+	1    5100 7450
 	1    0    0    -1
 $EndComp
@@
 	0    -1   -1   0
 $EndComp
-Text Label 6350 6800 2    50   ~ 0
+Text Label 5100 7450 2    50   ~ 0
 5V_EN_L
+Text Label 2600 5150 0    50   ~ 0
+SDA
+Text Label 2600 4550 0    50   ~ 0
+SCL
+Wire Wire Line
+	9150 3800 8850 3800
+Text Label 9500 4350 2    50   ~ 0
+SDO
+$Comp
+L Device:R_Small_US R12
+U 1 1 61B27D5C
+P 9150 3900
+F 0 "R12" H 9218 3946 50  0000 L CNN
+F 1 "10K" H 9218 3855 50  0000 L CNN
+F 2 "Resistor_SMD:R_0402_1005Metric" H 9150 3900 50  0001 C CNN
+F 3 "~" H 9150 3900 50  0001 C CNN
+	1    9150 3900
+	1    0    0    -1
+$EndComp
+Text Label 9150 4100 0    50   ~ 0
+SDO
+Wire Wire Line
+	9150 4100 9150 4000
+Text Label 2600 4950 0    50   ~ 0
+FIRE_L
+$Comp
+L power:GND #PWR0148
+U 1 1 61B7977C
+P 6100 7350
+F 0 "#PWR0148" H 6100 7100 50  0001 C CNN
+F 1 "GND" H 6105 7177 50  0000 C CNN
+F 2 "" H 6100 7350 50  0001 C CNN
+F 3 "" H 6100 7350 50  0001 C CNN
+	1    6100 7350
+	1    0    0    -1
+$EndComp
+$Comp
+L Device:R_Small_US R21
+U 1 1 61B79FEE
+P 6100 7250
+F 0 "R21" H 6168 7296 50  0000 L CNN
+F 1 "100K" H 6168 7205 50  0000 L CNN
+F 2 "Resistor_SMD:R_0402_1005Metric" H 6100 7250 50  0001 C CNN
+F 3 "~" H 6100 7250 50  0001 C CNN
+	1    6100 7250
+	1    0    0    -1
+$EndComp
+$Comp
+L Device:R_Small_US R16
+U 1 1 61B8E8A6
+P 6100 7050
+F 0 "R16" H 6168 7096 50  0000 L CNN
+F 1 "100K" H 6168 7005 50  0000 L CNN
+F 2 "Resistor_SMD:R_0402_1005Metric" H 6100 7050 50  0001 C CNN
+F 3 "~" H 6100 7050 50  0001 C CNN
+	1    6100 7050
+	1    0    0    -1
+$EndComp
+$Comp
+L power:+BATT #PWR0149
+U 1 1 61B987D5
+P 6100 6950
+F 0 "#PWR0149" H 6100 6800 50  0001 C CNN
+F 1 "+BATT" V 6115 7077 50  0000 L CNN
+F 2 "" H 6100 6950 50  0001 C CNN
+F 3 "" H 6100 6950 50  0001 C CNN
+	1    6100 6950
+	1    0    0    -1
+$EndComp
+Text Label 6400 7150 0    50   ~ 0
+BAT_VSENSE
+$Comp
+L Device:R_Small_US R17
+U 1 1 61B52924
+P 3150 1000
+F 0 "R17" V 2945 1000 50  0000 C CNN
+F 1 "10K" V 3036 1000 50  0000 C CNN
+F 2 "Resistor_SMD:R_0402_1005Metric" H 3150 1000 50  0001 C CNN
+F 3 "~" H 3150 1000 50  0001 C CNN
+	1    3150 1000
+	1    0    0    1
+$EndComp
+Wire Wire Line
+	3150 1300 3150 1100
+Wire Wire Line
+	3150 900  3150 700
+Connection ~ 3150 700
+Wire Wire Line
+	3150 700  4050 700
+Text Label 2600 6050 0    50   ~ 0
+CHARGE_CAP_EN
+Text Label 2600 6350 0    50   ~ 0
+BAT_VSENSE
+$Comp
+L power:GND #PWR0150
+U 1 1 61C1ECC9
+P 2550 1700
+F 0 "#PWR0150" H 2550 1450 50  0001 C CNN
+F 1 "GND" H 2555 1527 50  0000 C CNN
+F 2 "" H 2550 1700 50  0001 C CNN
+F 3 "" H 2550 1700 50  0001 C CNN
+	1    2550 1700
+	1    0    0    -1
+$EndComp
+$Comp
+L Device:R_Small_US R23
+U 1 1 61C1ECCF
+P 2550 1600
+F 0 "R23" H 2618 1646 50  0000 L CNN
+F 1 "100K" H 2618 1555 50  0000 L CNN
+F 2 "Resistor_SMD:R_0402_1005Metric" H 2550 1600 50  0001 C CNN
+F 3 "~" H 2550 1600 50  0001 C CNN
+	1    2550 1600
+	1    0    0    -1
+$EndComp
+$Comp
+L Device:R_Small_US R22
+U 1 1 61C1ECD5
+P 2550 1400
+F 0 "R22" H 2618 1446 50  0000 L CNN
+F 1 "100K" H 2618 1355 50  0000 L CNN
+F 2 "Resistor_SMD:R_0402_1005Metric" H 2550 1400 50  0001 C CNN
+F 3 "~" H 2550 1400 50  0001 C CNN
+	1    2550 1400
+	1    0    0    -1
+$EndComp
+Wire Wire Line
+	6400 7150 6100 7150
+Connection ~ 6100 7150
+Text Label 2800 1500 0    50   ~ 0
+CAP_VSENSE
+Wire Wire Line
+	2800 1500 2550 1500
+Connection ~ 2550 1500
+Text Label 2600 4750 0    50   ~ 0
+CAP_VSENSE
+Wire Wire Line
+	2600 4850 3050 4850
+Connection ~ 2550 1300
+Wire Wire Line
+	2550 1300 2750 1300
+Text Label 2600 5950 0    50   ~ 0
+BCLK
+Text Label 2600 6250 0    50   ~ 0
+D_OUT_I2S
+Text Label 2600 5850 0    50   ~ 0
+WS
 $EndSCHEMATC
